Commit message: minor fixes

File: softgripper_description/urdf/softgripper.xacro (robot description, xacro)
@@ -5,5 +5,5 @@
     <!-- Link to world -->
     <joint name="base_joint" type="fixed">
-        <origin xyz="0 0 0" rpy="0 0 0"/>
+        <origin xyz="0 0 0" rpy="0 -1.5708 0"/>
         <parent link="world"/>
         <child link="flange" />
